Commit message: add a urdf file of the 2022 HERO

File: src/test/urdf/test.urdf (robot description, URDF)
Before this commit: robot test, 7 links, 6 joints
Links:
- link Left_back_link: mass 0.6407 -> 0.640701994677817
- link Left_front_Link: mass 0.59406 -> 0.59406052726133
- link Pitch_link: mass 0 -> 2.47332642999639
- link Right_back_link: mass 0.59406 -> 0.594060518100536
- link Right_front_link: mass 0.6407 -> 0.640702005693192
- link Yaw_link: mass 0.48017 -> 0.480169882095531
Joints:
- joint Left_front_joint: axis 0 0 1 -> 1 0 0
- joint Pitch_joint: origin xyz=0 0 0.238 rpy=0 0 0 -> xyz=-0.0456 -0.02439 0.07757 rpy=0 0 0; parent base_link -> Yaw_link
- joint Right_front_link: axis 0 0 1 -> -1 0 0

Commit message: refine the urdf file to enable the gazebo simulation

File: src/test/urdf/test.urdf (robot description, URDF)
Before this commit: robot test, 7 links, 6 joints
Links:
- added link base_foot_print
Joints:
- removed joint Right_front_link
- removed joint Yaw_link
- added joint Right_front_joint: type continuous, parent base_link, child Right_front_link, origin xyz=-0.2345 -0.22007 -0.028122 rpy=0 0 0, axis -1 0 0
- added joint Yaw_joint: type continuous, parent base_link, child Yaw_link, origin xyz=0 0 0.238 rpy=0 0 0, axis 0 0 -1
- added joint base_foot_print_joint: type fixed, parent base_foot_print, child base_link, origin xyz=0 0 0.2 rpy=0 0 3.14, axis 1 0 0
